File: Adafruit Feather RP2040 Original.brd (EAGLE design)
At the start: 50.8 x 22.9 mm, 61 parts, among them IC1 RP2040_QFN56, Q3 DMG3415, SW1 KMR2, SW3 Mini RA Switch, U1 W25Q64JVSSIQ, U2 RT9080/AP2112-3.3, U3 MCP73831T-2ACI/OT, X1 JSTPH, X2 2x5 SWD, X6 USB Type C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

Commit message: Add new rev.
Parts:
- removed D1: NSR0320, microbuilder:SOD-323_MINI
- removed SW3: Mini RA Switch, adafruit_electromech:SPST_TACTILE_RA_2*4*3.5MM
- added SW2: KMR2, microbuilder:BTN_KMR2_4.6X2.8
- C1, C20, C4: value 10uF -> 10µF
- CONN1: device adafruit_electromech:JST_SH4 -> microbuilder:JST_SH4
- D4: value MBR0540 -> MBR540
- Q3: value DMG3415 -> DMG341
- SW1: device adafruit_electromech:BTN_KMR2_4.6X2.8 -> microbuilder:BTN_KMR2_4.6X2.8
- U$31, U$32: device adafruit_electromech:MOUNTINGHOLE_2.5_PLATED -> microbuilder:MOUNTINGHOLE_2.5_PLATED
- U1: value W25Q64JVSSIQ -> 2MB Flash; device microbuilder:USON8_4X4 -> microbuilder:SOIC8_208MIL
- U2: value RT9080/AP2112-3.3 -> AP2112-3.3; device adafruit_power:SOT23-5 -> microbuilder:SOT23-5@1
- X1: device adafruit_electromech:JSTPH2_BATT -> microbuilder:JSTPH2_BATT
- X2: value 2x5 SWD -> (none); device adafruit_electromech:2X05_1.27MM_BOX_NOCREAM -> microbuilder:2X05_1.27MM_BOX_POSTS
- X6: device adafruit_electromech:USB_C_CUSB31-CFM2AX-01-X -> microbuilder:USB_C_CUSB31-CFM2AX-01-X
- Y1: value 12MHz/12pF -> 12MHZ
- moved X1 1.65 mm to (10.9, 19.3)
- moved X6 1.27 mm to (2.60, 11.4)
- moved C15 0.77 mm to (37.8, 17.5), turned to 180 degrees
- moved U1 0.74 mm to (42.3, 14.7), turned to 180 degrees
- moved C14 0.51 mm to (34.0, 17.7)
- moved CONN1 0.51 mm to (48.3, 8.26)
- moved R5 0.46 mm to (45.4, 13.3)
- moved R11 0.40 mm to (45.3, 16.3)
Connections:
- removed net N$8: D1.A, R11.2
- net GND: now also SW2.B, SW2.B'; no longer SW3.1, SW3.MT1, SW3.MT2, U1.PAD, X1.NC1, X1.NC2
- net USBBOOT: now also R11.2, SW2.A, SW2.A'; no longer D1.C, IC1.6, SW3.2
Routing:
- net USBBOOT: track 24.5 -> 10.0 mm, vias 3 -> 1
- net GND: track 37.2 -> 29.3 mm, vias 41 -> 40
- net QSPI_DATA[0]: track 3.24 -> 10.5 mm, vias 0 -> 2
- net QSPI_SCK: track 4.66 -> 11.4 mm, vias 0 -> 2
- net QSPI_CS: track 11.7 -> 17.3 mm
- net QSPI_DATA[1]: track 7.25 -> 11.0 mm
- net N$8: track 1.68 -> 0.00 mm
- net QSPI_DATA[2]: track 6.29 -> 7.72 mm
- net D-: track 45.6 -> 44.6 mm
- net QSPI_DATA[3]: track 5.78 -> 6.43 mm
- net SCL: track 25.3 -> 24.7 mm
- net +3V3: track 115.5 -> 114.9 mm
- net 1.2V: track 22.5 -> 21.9 mm
- net D6: track 10.4 -> 9.87 mm
Other:
- board text removed: "8MB"
