File: Adafruit Feather RP2040.sch (EAGLE design)
At the start: 57 parts, among them IC1 RP2040_QFN56, Q3 DMG341, SW1 KMR2, SW2 KMR2, U1 2MB Flash, U2 AP2112-3.3, U3 MCP73831T-2ACI/OT, X1 JSTPH, X6 USB Type C, Y1 12MHZ

Commit message: Add new rev.
Parts:
- removed SW2: KMR2, microbuilder:SWITCH_TACT_SMT4.6X2.8
- added D1: NSR0320, microbuilder:DIODE_SOD323MINI
- added SW3: Mini RA Switch, adafruit_electromech:SWITCH_SPST_MNT_2*4*3.5
- C1, C20: value 10µF -> 10uF
- C4: value 10µF -> 10uF; REV C -> D
- CONN1: device microbuilder:STEMMA_I2C_QT -> adafruit_electromech:STEMMA_I2C_QT
- D4: value MBR540 -> MBR0540
- Q3: value DMG341 -> DMG3415
- SW1: device microbuilder:SWITCH_TACT_SMT4.6X2.8 -> adafruit_electromech:SWITCH_TACT_SMT4.6X2.8
- U$31, U$32: device microbuilder:MOUNTINGHOLE2.5 -> adafruit_electromech:MOUNTINGHOLE2.5
- U1: value 2MB Flash -> W25Q64JVSSIQ; device microbuilder:SPIFLASH_8PIN208MIL -> microbuilder:SPIFLASH_8PIN_4X4
- U2: value AP2112-3.3 -> RT9080/AP2112-3.3; device microbuilder:VREG_SOT23-5 -> adafruit_power:VREG_SOT23-5; JLC_ROTATION (none) -> 0
- X1: device microbuilder:CON_JST_PH_2PIN_BATT -> adafruit_electromech:CON_JST_PH_2PIN_MT_BATT
- X2: value (none) -> 2x5 SWD; device microbuilder:JTAG-CORTEXBOXPOSTS -> adafruit_electromech:JTAG-CORTEX_NOCREAM
- X6: device microbuilder:USB_C -> adafruit_electromech:USB_C
- Y1: value 12MHZ -> 12MHz/12pF
Connections:
- new net N$8: D1.A, R11.2
- net GND: now also SW3G$1.P, SW3G$2.MT, X1G$1.1, X1MT1.P$1, X1MT2.P$1; no longer SW2.S, SW2.S1, X1.1
- net USBBOOT: now also D1.C, IC1.GPIO4, SW3G$1.S; no longer R11.2, SW2.P, SW2.P1
- net VBAT: now also X1G$1.2; no longer X1.2
Other:
- moved on the sheet: R11, U1
